Commit message: navigation is working but not dynamic

File: src/my_robot_description/urdf/robot.urdf (robot description, URDF)
Before this commit: robot mechatronics_robot, 5 links, 4 joints
Links:
- removed link caster_wheel
- added link base_footprint
- added link camera_link; visual box size=0.02 0.05 0.02
- added link gps_link; visual cylinder length=0.01 radius=0.03
- added link imu_link; visual box size=0.02 0.02 0.01
- link base_link: mass 5.0 -> 10.0; geometry collision box size=0.6 0.4 0.1; visual box size=0.6 0.4 0.1
- link left_wheel: mass 0.5 -> 2.0
- link livox_frame: mass 0.2 -> None; geometry visual cylinder length=0.04 radius=0.05
- link right_wheel: mass 0.5 -> 2.0
Joints:
- removed joint caster_joint
- removed joint livox_joint
- added joint base_joint: type fixed, parent base_footprint, child base_link, origin xyz=0 0 0.10 rpy=0 0 0
- added joint camera_joint: type fixed, parent base_link, child camera_link, origin xyz=0.3 0 0.08 rpy=0 0 0
- added joint gps_joint: type fixed, parent base_link, child gps_link, origin xyz=-0.25 0 0.12 rpy=0 0 0
- added joint imu_joint: type fixed, parent base_link, child imu_link, origin xyz=0 0 0.05 rpy=0 0 0
- added joint lidar_joint: type fixed, parent base_link, child livox_frame, origin xyz=0 0 0.12 rpy=0 0 0
- joint left_wheel_joint: origin xyz=0.15 0.225 -0.05 rpy=-1.5708 0 0 -> xyz=0 0.225 0 rpy=-1.5708 0 0
- joint right_wheel_joint: origin xyz=0.15 -0.225 -0.05 rpy=-1.5708 0 0 -> xyz=0 -0.225 0 rpy=-1.5708 0 0

Commit message: every thing is working but need to optimize

File: src/my_robot_description/urdf/robot.urdf (robot description, URDF)
Before this commit: robot my_robot, 7 links, 6 joints
Links:
- link livox_frame: geometry visual cylinder length=0.05 radius=0.05
Joints:
- joint lidar_joint: origin xyz=0 0 0.12 rpy=0 0 0 -> xyz=0 0 0.13 rpy=0 0 0
